File: hackpads/coolhackpad/pcb/HackPad.kicad_pcb (KiCad board)
At the start: 2 copper layers, 99.5 x 85 mm, 37 parts, among them SW1 SW_Push, SW10 SW_Push, SW11 SW_Push, SW12 SW_Push, SW13 SW_Push, SW14 SW_Push, SW15 SW_Push, SW16 SW_Push, SW17 RotaryEncoder, SW2 SW_Push, SW3 SW_Push, SW4 SW_Push, SW5 SW_Push, SW6 SW_Push, SW7 SW_Push, SW8 SW_Push, SW9 SW_Push, U1 SeeeduinoXIAO

Commit message: update PCB
Parts:
- removed U1: SeeeduinoXIAO, Seeed Studio XIAO Series Library:XIAO-Generic-Thruhole-14P-2.54-21X17.8MM
- added R1: 10k, Resistor_THT:R_Axial_DIN0207_L6.3mm_D2.5mm_P7.62mm_Horizontal, F.Cu at (114.5, 66.3)
- added U2: Seeed Studio XIAO SAMD21, Seeed Studio XIAO Series Library:XIAO-Generic-Thruhole-14P-2.54-21X17.8MM, F.Cu at (120.4, 29.0)
- SW17: value RotaryEncoder -> RotaryEncoder_Switch; footprint Rotary_Encoder:RotaryEncoder_Alps_EC11E_Vertical_H20mm -> Rotary_Encoder:RotaryEncoder_Alps_EC11E-Switch_Vertical_H20mm
- moved SW16 39.0 mm to (101.5, 80.4)
- moved SW2 39.0 mm to (44.5, 42.4)
- moved SW6 39.0 mm to (63.5, 42.4)
- moved D1 39.0 mm to (51.5, 32.0)
- moved D10 39.0 mm to (89.5, 51.3)
- moved D11 39.0 mm to (89.5, 69.8)
- moved D12 39.0 mm to (89.5, 88.6)
- moved D13 39.0 mm to (108.5, 32.1)
- moved D14 39.0 mm to (108.5, 51.1)
- moved D15 39.0 mm to (108.5, 70.1)
- moved D16 39.0 mm to (108.5, 88.6)
- moved D2 39.0 mm to (51.5, 51.3)
- moved D3 39.0 mm to (51.5, 70.3)
- moved D4 39.0 mm to (51.5, 88.6)
- moved D5 39.0 mm to (70.5, 32.1)
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- renumbered REF** to M2.5
Routing:
- net +3.3V: track 0.00 -> 39.9 mm
- net GND: track 30.8 -> 0.00 mm
- net Net-(R1-Pad1): track 0.00 -> 21.7 mm
- net A10: track 0.00 -> 18.4 mm
- net A9: track 24.6 -> 20.3 mm
- net A8: track 26.2 -> 23.9 mm
- added copper zone on B.Cu, net GND
Other:
- board size 99.5 x 85 mm -> 99.5 x 86 mm
- board text added: "Made in 2024 By Zhixuan"
- board text added: "Thx project HackPad"
- board text removed: "Made by Zhixuan. In 2024."
- board text removed: "Thx project HackPad!"
