File: hackpads/nimit/pcb/nimitpad.kicad_pcb (KiCad board)
At the start: 2 copper layers, 99.1 x 99.1 mm, 26 parts, among them J1 Conn_01x04, M1 XIAO-RP2040, SW1 RotaryEncoder_Switch, SW10 SW_Push, SW11 SW_Push, SW12 SW_Push, SW2 SW_Push, SW3 SW_Push, SW4 SW_Push, SW5 SW_Push, SW6 SW_Push, SW7 SW_Push, SW8 SW_Push, SW9 SW_Push

Commit message: Update nimitpad.kicad_pcb
Parts:
- J1: footprint Library:128x64OLED -> Connector_PinHeader_2.54mm:PinHeader_1x04_P2.54mm_Vertical
- SW1: footprint Rotary_Encoder:RotaryEncoder_Alps_EC11E-Switch_Vertical_H20mm -> Rotary_Encoder:EC11E
- moved J1 16.7 mm to (45.7, 72.4), turned to -90 degrees
- moved SW1 0.46 mm to (64.9, 41.9)
Routing:
- net Net-(J1-Pin_2): track 33.4 -> 9.67 mm, vias 1 -> 0
- net Net-(J1-Pin_1): track 34.7 -> 13.3 mm
- net Net-(J1-Pin_3): track 47.7 -> 36.9 mm
- net Net-(J1-Pin_4): track 80.1 -> 73.0 mm
- net Net-(D1-A): track 7.97 -> 9.50 mm
