File: hackpads/Soup-Pad/pcb/keypad.kicad_pcb (KiCad board)
At the start: 2 copper layers, 88.9 x 150 mm, 73 parts, among them J2 VL53L0X, J3 DHT11, M2 MOUDLE-SEEEDUINO-XIAO, SW1 SW_Push_45deg, SW10 SW_Push_45deg, SW11 SW_Push_45deg, SW12 SW_Push_45deg, SW15 RotaryEncoder_Switch, SW16 RotaryEncoder_Switch, SW2 SW_Push_45deg, SW3 SW_Push_45deg, SW4 SW_Push_45deg, SW5 SW_Push_45deg, SW6 SW_Push_45deg, SW7 SW_Push_45deg, SW8 SW_Push_45deg, SW9 SW_Push_45deg, U1 MCP23008-xSO

Commit message: Add files via upload
Routing:
- net GND: track 778.4 -> 772.4 mm, vias 30 -> 29
- net ENC_SW1: track 95.2 -> 95.3 mm, vias 4 -> 5
Changed lines of the file:
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@@
 	)
 	(gr_text "Souptik"
-		(at 137.5 90.5 -0)
+		(at 137.5 90.5 0)
 		(layer "B.SilkS")
 		(effects
@@
 			(justify left bottom mirror)
 		)
-		(render_cache "Souptik" -0
+		(render_cache "Souptik" 0
 			(polygon
 				(pts
@@
 	)
 	(gr_text "Souptik\n"
-		(at 124.75 69 0)
-		(layer "Edge.Cuts")
+		(at 140.6 90.6 0)
+		(layer "F.SilkS")
 		(effects
 			(font
@@
 	)
 	(gr_text "Souptik\n"
-		(at 132.5 90.75 0)
+		(at 124.75 69 0)
 		(layer "Edge.Cuts")
 		(effects
@@
 	)
 	(segment
+		(start 160.6 140.6)
+		(end 160.59 140.59)
+		(width 0.2)
+		(layer "F.Cu")
+		(net 1)
+	)
+	(segment
 		(start 90.26 138.76)
 		(end 90.26 141.225)
@@
 	)
 	(segment
+		(start 160.59 140.59)
+		(end 158.84 140.59)
+		(width 0.2)
+		(layer "F.Cu")
+		(net 1)
+	)
+	(segment
 		(start 165.25 88.5)
 		(end 168.25 88.5)
@@
 	)
 	(segment
-		(start 158.84 139.91)
-		(end 160.75 138)
-		(width 0.2)
-		(layer "F.Cu")
-		(net 1)
-	)
-	(segment
 		(start 137.7 164.56)
 		(end 138.43 163.83)
@@
 	)
 	(segment
-		(start 158.84 140.59)
-		(end 158.84 139.91)
-		(width 0.2)
-		(layer "F.Cu")
-		(net 1)
-	)
-	(segment
 		(start 160.02 163.83)
 		(end 165.735 163.83)
@@
 	)
 	(via
-		(at 168.25 138)
-		(size 0.6)
-		(drill 0.3)
-		(layers "F.Cu" "B.Cu")
-		(net 1)
-	)
-	(via
 		(at 150.85 49.25)
 		(size 0.6)
@@
 	)
 	(via
-		(at 160.75 138)
+		(at 151.765 163.83)
 		(size 0.6)
 		(drill 0.3)
@@
 	)
 	(via
-		(at 151.765 163.83)
+		(at 146.685 163.83)
 		(size 0.6)
 		(drill 0.3)
@@
 	)
 	(via
-		(at 146.685 163.83)
+		(at 165.25 88.5)
 		(size 0.6)
 		(drill 0.3)
@@
 	)
 	(via
-		(at 165.25 88.5)
+		(at 98.75 49.75)
 		(size 0.6)
 		(drill 0.3)
@@
 	)
 	(via
-		(at 98.75 49.75)
+		(at 84.85 75.5)
 		(size 0.6)
 		(drill 0.3)
@@
 	)
 	(via
-		(at 84.85 75.5)
+		(at 160.6 140.6)
 		(size 0.6)
 		(drill 0.3)
@@
 	)
 	(segment
+		(start 161.19 140.59)
+		(end 163.74 140.59)
+		(width 0.2)
+		(layer "B.Cu")
+		(net 1)
+	)
+	(segment
 		(start 93.345 72.425)
 		(end 93.345 71.995)
@@
 	)
 	(segment
+		(start 161.18 140.6)
+		(end 161.19 140.59)
+		(width 0.2)
+		(layer "B.Cu")
+		(net 1)
+	)
+	(segment
 		(start 90.26 138.74)
 		(end 90.25 138.75)
@@
 	)
 	(segment
-		(start 160.75 138)
-		(end 168.25 138)
+		(start 160.6 140.6)
+		(end 161.18 140.6)
 		(width 0.2)
 		(layer "B.Cu")
@@
 	)
 	(segment
+		(start 137.4 56.4)
+		(end 137.263 56.537)
+		(width 0.2)
+		(layer "F.Cu")
+		(net 56)
+	)
+	(segment
 		(start 111.76 84.455)
 		(end 118.11 84.455)
@@
 		(net 56)
 	)
+	(segment
+		(start 137.263 56.537)
+		(end 134.6175 56.537)
+		(width 0.2)
+		(layer "F.Cu")
+		(net 56)
+	)
 	(via
 		(at 142.24 56.515)
@@
 	)
 	(via
+		(at 137.4 56.4)
+		(size 0.6)
+		(drill 0.3)
+		(layers "F.Cu" "B.Cu")
+		(net 56)
+	)
+	(via
 		(at 111.76 84.455)
 		(size 0.6)
@@
 	)
 	(segment
-		(start 136.503 56.537)
-		(end 136.525 56.515)
+		(start 137.4 56.4)
+		(end 137.515 56.515)
 		(width 0.2)
 		(layer "B.Cu")
@@
 	)
 	(segment
-		(start 142.24 84.455)
-		(end 142.24 76.835)
+		(start 137.515 56.515)
+		(end 142.24 56.515)
 		(width 0.2)
 		(layer "B.Cu")
@@
 	)
 	(segment
-		(start 142.24 56.515)
-		(end 134.6395 56.515)
+		(start 142.24 84.455)
+		(end 142.24 76.835)
 		(width 0.2)
 		(layer "B.Cu")
@@
 		(hatch edge 0.5)
 		(connect_pads
-			(clearance 1)
+			(clearance 0.6)
 		)
 		(min_thickness 0.6)
