File: hackpads/hajpad/pcb/macropad.kicad_pcb (KiCad board)
At the start: 2 copper layers, 99 x 99 mm, 32 parts, among them SW1 RotaryEncoder_Switch, SW10 SW_Push_45deg, SW2 SW_Push_45deg, SW3 SW_Push_45deg, SW4 SW_Push_45deg, SW5 SW_Push_45deg, SW6 SW_Push_45deg, SW7 SW_Push_45deg, SW8 SW_Push_45deg, SW9 SW_Push_45deg, U1 Seeed Studio XIAO SAMD21

Commit message: added astolpho and date yippeeeee
Parts:
- added G***: LOGO, LOGO, B.Cu at (176.8, 130.4)
Other:
- board text added: "AH FUCK MY SHOULDERS"
- board text added: "October 2024 :3"
