File: hackpads/Ctrl_pad/pcb/Ctrl_pad.kicad_pcb (KiCad board)
At the start: 2 copper layers, 62.5 x 100 mm, 23 parts, among them J1 0.96" OLED Display, SW1 MX, SW2 MX, SW3 MX, SW4 MX, SW5 MX, SW6 MX, SW7 RotaryEncoder_Switch, SW8 MX, SW9 MX, U1 MCU_Seeed_XIAO_RP2040

Commit message: Update PCB
Parts:
- J1: footprint Display:Adafruit_SSD1306 -> ScottoKeebs_Components:OLED_128x64
- moved J1 10.6 mm to (138.2, 59.5)
Routing:
- net GND: track 65.3 -> 74.0 mm
- net SCL: track 75.5 -> 81.8 mm
- net +3.3V: track 71.6 -> 77.3 mm
- net SDA: track 79.7 -> 81.0 mm
