File: hackpads/Ctrl_pad/pcb/Ctrl_pad.kicad_sch (KiCad schematic)
At the start: 22 parts, among them J1 0.96" OLED Display, SW1 MX, SW2 MX, SW3 MX, SW4 MX, SW5 MX, SW6 MX, SW7 RotaryEncoder_Switch, SW8 MX, SW9 MX, U1 MCU_Seeed_XIAO_RP2040

Commit message: Update PCB
Parts:
- J1: footprint Display:Adafruit_SSD1306 -> ScottoKeebs_Components:OLED_128x64
Changed lines of the file:
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@@
 			)
 		)
-		(property "Footprint" "Display:Adafruit_SSD1306"
+		(property "Footprint" "ScottoKeebs_Components:OLED_128x64"
 			(at 209.55 41.91 0)
 			(effects
