File: hackpads/MiniGamePad/pcb/HackPad.kicad_pcb (KiCad board)
At the start: 2 copper layers, 100 x 69 mm, 36 parts, among them J1 OLED_128x64, SW1 SW_Push_45deg, SW10 RotaryEncoder_Switch, SW2 SW_Push_45deg, SW3 SW_Push_45deg, SW4 SW_Push_45deg, SW5 SW_Push_45deg, SW6 SW_Push_45deg, SW7 SW_Push_45deg, SW8 SW_Push_45deg, U1 MOUDLE-SEEEDUINO-XIAO

Commit message: change text on the board
Other:
- board text added: "MINIGAME-PAD"
- board text removed: "GAMEPAD"
