File: hackpads/Kokary_HackPad/pcb/Schematic.kicad_pcb (KiCad board)
At the start: 2 copper layers, 6 parts, among them SW1 SW_Push, SW2 SW_Push, SW3 SW_Push, SW4 SW_Push, SW5 SW_Push, U1 Seeed Studio XIAO SAMD21

Commit message: modified:   hackpads/Kokary_HackPad/pcb/Schematic.kicad_pcb 	modified:   hackpads/Kokary_HackPad/pcb/Schematic.kicad_prl 	modified:   hackpads/Kokary_HackPad/pcb/Schematic.kicad_pro
Connections:
- net GND renamed row 0
- SW4 pad 1: Net-(U1-PA9_A5_D5_SCL) -> Net-(U1-PB08_A6_D6_TX)
- U1 pad 7: Net-(U1-PA9_A5_D5_SCL) -> Net-(U1-PB08_A6_D6_TX)
Routing:
- net Net-(U1-PA9_A5_D5_SCL): track 117.9 -> 70.6 mm
- net Net-(U1-PB08_A6_D6_TX): track 0.00 -> 47.3 mm
Changed lines of the file:
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@@
 	)
 	(net 0 "")
-	(net 1 "GND")
+	(net 1 "row 0")
 	(net 2 "Net-(U1-PA5_A9_D9_MISO)")
 	(net 3 "Net-(U1-PA6_A10_D10_MOSI)")
@@
 	(net 12 "unconnected-(U1-PB09_A7_D7_RX-Pad8)")
 	(net 13 "unconnected-(U1-5V-Pad14)")
+	(net 14 "Net-(U1-PB08_A6_D6_TX)")
 	(footprint "Button_Switch_Keyboard:SW_Cherry_MX_1.00u_PCB"
 		(layer "F.Cu")
@@
 			)
 		)
-		(sheetname "Stammblatt")
+		(sheetname "Root")
 		(sheetfile "Schematic.kicad_sch")
 		(attr through_hole)
@@
 			(layers "*.Cu" "*.Mask")
 			(remove_unused_layers no)
-			(net 1 "GND")
+			(net 1 "row 0")
 			(pinfunction "2")
 			(pintype "passive")
@@
 			)
 		)
-		(sheetname "Stammblatt")
+		(sheetname "Root")
 		(sheetfile "Schematic.kicad_sch")
 		(attr through_hole)
@@
 			(layers "*.Cu" "*.Mask")
 			(remove_unused_layers no)
-			(net 1 "GND")
+			(net 1 "row 0")
 			(pinfunction "2")
 			(pintype "passive")
@@
 			)
 		)
-		(sheetname "Stammblatt")
+		(sheetname "Root")
 		(sheetfile "Schematic.kicad_sch")
 		(attr through_hole)
@@
 			(layers "*.Cu" "*.Mask")
 			(remove_unused_layers no)
-			(net 1 "GND")
+			(net 1 "row 0")
 			(pinfunction "2")
 			(pintype "passive")
@@
 			)
 		)
-		(sheetname "Stammblatt")
+		(sheetname "Root")
 		(sheetfile "Schematic.kicad_sch")
 		(attr through_hole)
@@
 			(layers "*.Cu" "*.Mask")
 			(remove_unused_layers no)
-			(net 1 "GND")
+			(net 1 "row 0")
 			(pinfunction "2")
 			(pintype "passive")
@@
 			)
 		)
-		(sheetname "Stammblatt")
+		(sheetname "Root")
 		(sheetfile "Schematic.kicad_sch")
 		(attr through_hole)
@@
 			(layers "*.Cu" "*.Mask")
 			(remove_unused_layers no)
-			(net 7 "Net-(U1-PA9_A5_D5_SCL)")
+			(net 14 "Net-(U1-PB08_A6_D6_TX)")
 			(pinfunction "1")
 			(pintype "passive")
@@
 			(layers "*.Cu" "*.Mask")
 			(remove_unused_layers no)
-			(net 1 "GND")
+			(net 1 "row 0")
 			(pinfunction "2")
 			(pintype "passive")
@@
 			)
 		)
-		(sheetname "Stammblatt")
+		(sheetname "Root")
 		(sheetfile "Schematic.kicad_sch")
 		(attr smd)
@@
 			(layers "*.Cu" "*.Mask")
 			(remove_unused_layers no)
-			(net 7 "Net-(U1-PA9_A5_D5_SCL)")
+			(net 14 "Net-(U1-PB08_A6_D6_TX)")
 			(pinfunction "PB08_A6_D6_TX")
 			(pintype "unspecified")
@@
 			(layers "*.Cu" "*.Mask")
 			(remove_unused_layers no)
-			(net 1 "GND")
+			(net 1 "row 0")
 			(pinfunction "GND")
 			(pintype "unspecified")
@@
 	)
 	(segment
-		(start 123 99.5)
-		(end 123 89.04)
+		(start 123.5 102.5)
+		(end 124.5 101.5)
 		(width 0.2)
 		(layer "B.Cu")
@@
 	)
 	(segment
-		(start 123.5 102.5)
-		(end 124.5 101.5)
+		(start 118.12 147.54)
+		(end 123.66 142)
 		(width 0.2)
 		(layer "B.Cu")
@@
 	)
 	(segment
-		(start 118.5 116.5)
-		(end 119.5 116.5)
+		(start 124.5 101.5)
+		(end 124.5 86.5)
 		(width 0.2)
 		(layer "B.Cu")
@@
 	)
 	(segment
-		(start 118.12 147.54)
-		(end 123.66 142)
+		(start 123.5 142)
+		(end 123.5 102.5)
 		(width 0.2)
 		(layer "B.Cu")
@@
 	)
 	(segment
-		(start 120.5 102)
-		(end 123 99.5)
+		(start 124.5 86.5)
+		(end 123 86.5)
 		(width 0.2)
 		(layer "B.Cu")
@@
 	)
 	(segment
-		(start 119.5 116.5)
-		(end 120.5 115.5)
+		(start 118.04 152.92)
+		(end 118.04 147.54)
 		(width 0.2)
 		(layer "B.Cu")
@@
 	)
 	(segment
-		(start 124.5 101.5)
-		(end 124.5 86.5)
+		(start 123 99.5)
+		(end 123 89.04)
 		(width 0.2)
 		(layer "B.Cu")
-		(net 7)
+		(net 14)
 	)
 	(segment
-		(start 118.12 133.46)
-		(end 118.16 133.5)
+		(start 118.5 116.5)
+		(end 119.5 116.5)
 		(width 0.2)
 		(layer "B.Cu")
-		(net 7)
+		(net 14)
 	)
 	(segment
-		(start 123.5 142)
-		(end 123.5 102.5)
+		(start 120.5 102)
+		(end 123 99.5)
 		(width 0.2)
 		(layer "B.Cu")
-		(net 7)
+		(net 14)
 	)
 	(segment
-		(start 120.5 115.5)
-		(end 120.5 102)
+		(start 119.5 116.5)
+		(end 120.5 115.5)
 		(width 0.2)
 		(layer "B.Cu")
-		(net 7)
+		(net 14)
 	)
 	(segment
-		(start 124.5 86.5)
-		(end 123 86.5)
+		(start 118.12 133.46)
+		(end 118.16 133.5)
 		(width 0.2)
 		(layer "B.Cu")
-		(net 7)
+		(net 14)
+	)
+	(segment
+		(start 120.5 115.5)
+		(end 120.5 102)
+		(width 0.2)
+		(layer "B.Cu")
+		(net 14)
 	)
 	(segment
@@
 		(width 0.2)
 		(layer "B.Cu")
-		(net 7)
+		(net 14)
 	)
 	(segment
@@
 		(width 0.2)
 		(layer "B.Cu")
-		(net 7)
+		(net 14)
 	)
 	(segment
@@
 		(width 0.2)
 		(layer "B.Cu")
-		(net 7)
+		(net 14)
 	)
 	(segment
@@
 		(width 0.2)
 		(layer "B.Cu")
-		(net 7)
-	)
-	(segment
-		(start 118.04 152.92)
-		(end 118.04 147.54)
-		(width 0.2)
-		(layer "B.Cu")
-		(net 7)
+		(net 14)
 	)
 )
