File: hackpads/blahajpad/PCB/hackpad.kicad_pcb (KiCad board)
At the start: 2 copper layers, 87.6 x 134.6 mm, 66 parts, among them SW1 RotaryEncoder_Switch, U1 SEEED-XIAO, U2 MCP23017_SP

Commit message: Update PCB
Parts:
- removed REF** (x3): MountingHole_3.2mm_M3, MountingHole:MountingHole_3.2mm_M3
Routing:
- net GND: track 53.8 -> 66.9 mm, vias 1 -> 4
