File: hackpads/SpacePad_Submission/PCB/hackpad_pcb#3.kicad_pcb (KiCad board)
At the start: 2 copper layers, 81 x 85.7 mm, 25 parts, among them M1 XIAO-RP2040, SW1 SW_Push, SW10 SW_Push, SW11 SW_Push, SW12 SW_Push, SW2 SW_Push, SW3 SW_Push, SW4 SW_Push, SW5 SW_Push, SW6 SW_Push, SW7 SW_Push, SW8 SW_Push, SW9 SW_Push

Commit message: fixed pcb design
Routing:
- net Row 0: track 63.8 -> 93.4 mm, vias 0 -> 1
- net Row 2: track 137.9 -> 151.0 mm
- net Row 1: track 113.6 -> 125.2 mm
- net Col 3: track 105.5 -> 106.4 mm
Changed lines of the file:
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@@
 			(pintype "power_in")
 		)
-		(model "C:/Users/Sprex/AppData/Local/Programs/KiCad/8.0/share/kicad/3dmodels/seeed.3dshapes/Seeed Studio XIAO RP2040 v26.step"
+		(model "C:/Users/Sprex/Downloads/library.pretty/Xiao RP2040 with pins v1.step"
 			(offset
-				(xyz 0 0 0)
+				(xyz 0 0 2.6)
 			)
 			(scale
@@
 	)
 	(segment
-		(start 105.41 60.0125)
-		(end 105.41 62.7901)
+		(start 99.356598 78.55)
+		(end 95.12 82.786598)
 		(width 0.2)
 		(layer "F.Cu")
@@
 	)
 	(segment
-		(start 95.12 93.363402)
-		(end 99.781098 98.0245)
+		(start 95.12 82.786598)
+		(end 95.12 93.363402)
 		(width 0.2)
 		(layer "F.Cu")
@@
 	)
 	(segment
-		(start 104.499425 63.700675)
-		(end 95.12 73.080101)
+		(start 106.8 62.438846)
+		(end 111.036154 66.675)
 		(width 0.2)
 		(layer "F.Cu")
@@
 	)
 	(segment
-		(start 105.41 62.7901)
-		(end 104.499425 63.700675)
+		(start 111.1235 98.075)
+		(end 111.174 98.0245)
 		(width 0.2)
 		(layer "F.Cu")
@@
 	)
 	(segment
+		(start 109.805 98.075)
+		(end 111.1235 98.075)
+		(width 0.2)
+		(layer "F.Cu")
+		(net 2)
+	)
+	(segment
+		(start 105.41 60.0125)
+		(end 106.8 61.4025)
+		(width 0.2)
+		(layer "F.Cu")
+		(net 2)
+	)
+	(segment
+		(start 111.036154 66.675)
+		(end 101.525101 66.675)
+		(width 0.2)
+		(layer "F.Cu")
+		(net 2)
+	)
+	(segment
+		(start 106.8 61.4025)
+		(end 106.8 62.438846)
+		(width 0.2)
+		(layer "F.Cu")
+		(net 2)
+	)
+	(segment
 		(start 99.781098 98.0245)
 		(end 109.855 98.0245)
@@
 	)
 	(segment
-		(start 95.12 82.786598)
-		(end 95.12 93.363402)
+		(start 95.12 73.080101)
+		(end 95.12 74.313402)
 		(width 0.2)
 		(layer "F.Cu")
@@
 	)
 	(segment
-		(start 128.905 98.0245)
-		(end 111.174 98.0245)
+		(start 95.12 93.363402)
+		(end 99.781098 98.0245)
 		(width 0.2)
 		(layer "F.Cu")
@@
 	)
 	(segment
-		(start 99.356598 78.55)
-		(end 95.12 82.786598)
+		(start 128.905 98.0245)
+		(end 111.174 98.0245)
 		(width 0.2)
 		(layer "F.Cu")
@@
 	)
 	(segment
-		(start 95.12 74.313402)
-		(end 99.356598 78.55)
+		(start 101.525101 66.675)
+		(end 95.12 73.080101)
 		(width 0.2)
 		(layer "F.Cu")
@@
 	)
 	(segment
-		(start 95.12 73.080101)
-		(end 95.12 74.313402)
+		(start 95.12 74.313402)
+		(end 99.356598 78.55)
 		(width 0.2)
 		(layer "F.Cu")
@@
 	)
 	(segment
+		(start 110.774 71.056837)
+		(end 111.436154 70.394683)
+		(width 0.2)
+		(layer "F.Cu")
+		(net 3)
+	)
+	(segment
+		(start 107.605 58.675)
+		(end 107.605 58.475)
+		(width 0.2)
+		(layer "F.Cu")
+		(net 3)
+	)
+	(segment
 		(start 109.855 78.9745)
 		(end 108.0325 77.152)
@@
 	)
 	(segment
+		(start 111.436154 61.922308)
+		(end 108.188846 58.675)
+		(width 0.2)
+		(layer "F.Cu")
+		(net 3)
+	)
+	(segment
+		(start 111.174 78.4555)
+		(end 111.174 78.9745)
+		(width 0.2)
+		(layer "F.Cu")
+		(net 3)
+	)
+	(segment
 		(start 167.005 78.9745)
 		(end 147.955 78.9745)
@@
 	)
 	(segment
+		(start 109.855 78.9745)
+		(end 110.774 78.0555)
+		(width 0.2)
+		(layer "F.Cu")
+		(net 3)
+	)
+	(segment
 		(start 128.905 78.9745)
 		(end 111.174 78.9745)
@@
 	)
 	(segment
+		(start 110.774 78.0555)
+		(end 111.174 78.4555)
+		(width 0.2)
+		(layer "F.Cu")
+		(net 3)
+	)
+	(segment
+		(start 111.436154 70.394683)
+		(end 111.436154 61.922308)
+		(width 0.2)
+		(layer "F.Cu")
+		(net 3)
+	)
+	(segment
+		(start 108.188846 58.675)
+		(end 107.605 58.675)
+		(width 0.2)
+		(layer "F.Cu")
+		(net 3)
+	)
+	(segment
+		(start 110.774 78.0555)
+		(end 110.774 71.056837)
+		(width 0.2)
+		(layer "F.Cu")
+		(net 3)
+	)
+	(via
+		(at 107.605 58.475)
+		(size 0.6)
+		(drill 0.3)
+		(layers "F.Cu" "B.Cu")
+		(net 3)
+	)
+	(segment
+		(start 107.605 58.475)
+		(end 104.4075 58.475)
+		(width 0.2)
+		(layer "B.Cu")
+		(net 3)
+	)
+	(segment
+		(start 104.4075 58.475)
+		(end 102.87 60.0125)
+		(width 0.2)
+		(layer "B.Cu")
+		(net 3)
+	)
+	(segment
 		(start 107.6325 73.66)
 		(end 109.855 71.4375)
@@
 	)
 	(segment
-		(start 106.85 58.9125)
-		(end 107.95 60.0125)
+		(start 109.855 117.0745)
+		(end 99.721556 117.0745)
 		(width 0.2)
 		(layer "F.Cu")
@@
 	)
 	(segment
-		(start 99.781098 117.0745)
-		(end 93.18625 110.479652)
+		(start 96.161154 57.475)
+		(end 105.4125 57.475)
 		(width 0.2)
 		(layer "F.Cu")
@@
 	)
 	(segment
-		(start 101.72 62.198846)
-		(end 101.72 59.586154)
+		(start 102.405 57.475)
+		(end 105.4125 57.475)
 		(width 0.2)
 		(layer "F.Cu")
@@
 	)
 	(segment
-		(start 109.855 117.0745)
-		(end 99.781098 117.0745)
+		(start 101.72 58.16)
+		(end 102.405 57.475)
+		(width 0.2)
+		(layer "F.Cu")
+		(net 5)
+	)
+	(segment
+		(start 99.721556 117.0745)
+		(end 94.05 111.402944)
+		(width 0.2)
+		(layer "F.Cu")
+		(net 5)
+	)
+	(segment
+		(start 101.72 62.198846)
+		(end 101.72 58.16)
 		(width 0.2)
 		(layer "F.Cu")
@@
 	)
 	(segment
-		(start 93.18625 70.732596)
-		(end 101.72 62.198846)
+		(start 94.05 59.586154)
+		(end 96.161154 57.475)
 		(width 0.2)
 		(layer "F.Cu")
@@
 	)
 	(segment
-		(start 102.393654 58.9125)
+		(start 105.4125 57.475)
 		(end 106.85 58.9125)
 		(width 0.2)
@@
 	)
 	(segment
-		(start 101.72 59.586154)
-		(end 102.393654 58.9125)
+		(start 147.955 117.0745)
+		(end 128.905 117.0745)
 		(width 0.2)
 		(layer "F.Cu")
@@
 	)
 	(segment
-		(start 147.955 117.0745)
-		(end 128.905 117.0745)
+		(start 94.05 111.402944)
+		(end 94.05 59.586154)
 		(width 0.2)
 		(layer "F.Cu")
@@
 	)
 	(segment
-		(start 93.18625 110.479652)
-		(end 93.18625 70.732596)
+		(start 106.85 58.9125)
+		(end 107.95 60.0125)
 		(width 0.2)
 		(layer "F.Cu")
@@
 	)
 	(segment
-		(start 108.426346 58.9125)
-		(end 102.393654 58.9125)
+		(start 103.431154 57.875)
+		(end 101.72 59.586154)
 		(width 0.2)
 		(layer "B.Cu")
@@
 	)
 	(segment
-		(start 101.72 61.4025)
-		(end 100.33 60.0125)
+		(start 113.2425 61.9125)
+		(end 109.205 57.875)
 		(width 0.2)
 		(layer "B.Cu")
@@
 	)
 	(segment
-		(start 111.426346 61.9125)
-		(end 108.426346 58.9125)
+		(start 160.02 90.17)
+		(end 160.02 71.12)
 		(width 0.2)
 		(layer "B.Cu")
@@
 	)
 	(segment
-		(start 160.02 71.12)
-		(end 150.8125 61.9125)
+		(start 109.205 57.875)
+		(end 103.431154 57.875)
 		(width 0.2)
 		(layer "B.Cu")
@@
 	)
 	(segment
-		(start 160.02 90.17)
-		(end 160.02 71.12)
+		(start 101.72 59.586154)
+		(end 101.72 61.4025)
 		(width 0.2)
 		(layer "B.Cu")
@@
 	)
 	(segment
-		(start 150.8125 61.9125)
-		(end 111.426346 61.9125)
+		(start 160.02 109.22)
+		(end 160.02 90.17)
 		(width 0.2)
 		(layer "B.Cu")
@@
 	)
 	(segment
-		(start 102.393654 58.9125)
-		(end 101.72 59.586154)
+		(start 160.02 71.12)
+		(end 150.8125 61.9125)
 		(width 0.2)
 		(layer "B.Cu")
@@
 	)
 	(segment
-		(start 160.02 109.22)
-		(end 160.02 90.17)
+		(start 150.8125 61.9125)
+		(end 113.2425 61.9125)
 		(width 0.2)
 		(layer "B.Cu")
@@
 	)
 	(segment
-		(start 101.72 59.586154)
-		(end 101.72 61.4025)
+		(start 101.72 61.4025)
+		(end 100.33 60.0125)
 		(width 0.2)
 		(layer "B.Cu")
