File: hackpads/BeliçBoard/pcb/hecpad.kicad_pcb (KiCad board)
At the start: 2 copper layers, 77.5 x 50.5 mm, 14 parts, among them J1 OLED_DISPLAY, SW1 SW_Push_45deg, SW2 SW_Push_45deg, SW3 SW_Push_45deg, SW4 SW_Push_45deg, SW5 RotaryEncoder_Switch, SW6 RotaryEncoder_Switch, U1 MOUDLE-SEEEDUINO-XIAO

Commit message: Add files via upload
Routing:
- net Net-(U1-PA5_A9_D9_MISO): track 95.8 -> 76.9 mm
- net Net-(J1-Pin_2): track 49.3 -> 33.8 mm, vias 2 -> 1
- net Net-(D6-A): track 45.9 -> 35.4 mm, vias 1 -> 0
- net Net-(D2-A): track 64.3 -> 53.9 mm, vias 2 -> 1
- net Net-(J1-Pin_1): track 40.9 -> 33.1 mm, vias 2 -> 1
- net Net-(U1-PA02_A0_D0): track 73.6 -> 68.0 mm, vias 2 -> 1
- net Net-(U1-PB09_A7_D7_RX): track 41.0 -> 37.2 mm
- net Net-(D1-A): track 59.8 -> 56.8 mm, vias 2 -> 1
- net Net-(U1-PA10_A2_D2): track 58.8 -> 60.2 mm
- net Net-(D3-A): track 66.1 -> 65.6 mm
