File: hackpads/yanpad/PCB/yanpad.kicad_pcb (KiCad board)
At the start: 2 copper layers, 94.5 x 59 mm, 23 parts, among them SW1 SW_Push, SW2 SW_Push, SW3 SW_Push, SW4 SW_Push, SW5 SW_Push, SW6 SW_Push, SW7 SW_Push, SW8 SW_Push, SW9 SW_Push, U1 XIAO-RP2040-DIP

Commit message: oops forgot the branding text stuff
Other:
- board text added: "YanPad"
Changed lines of the file:
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@@
 		(layer "Edge.Cuts")
+	)
+	(gr_text "YanPad"
+		(at 112.5 121.5 0)
+		(layer "B.SilkS")
+		(effects
+			(font
+				(size 1 1)
+				(thickness 0.1)
+			)
+			(justify left bottom mirror)
+		)
 	)
 	(gr_text "XIAO HERE!"
