File: hackpads/N0PAD/pcb/N0PAD.kicad_pcb (KiCad board)
At the start: 2 copper layers, 93.5 x 98 mm, 38 parts, among them SW1 SW_Push_45deg, SW10 SW_Push_45deg, SW11 SW_Push_45deg, SW12 SW_Push_45deg, SW13 SW_Push_45deg, SW14 SW_Push_45deg, SW15 RotaryEncoder_Switch, SW2 SW_Push_45deg, SW3 SW_Push_45deg, SW4 SW_Push_45deg, SW5 SW_Push_45deg, SW6 SW_Push_45deg, SW7 SW_Push_45deg, SW8 SW_Push_45deg, SW9 SW_Push_45deg, U1 Seeed Studio XIAO RP2040

Commit message: more pcb files
Parts:
- moved G*** 1.00 mm to (158.5, 56.0)
- moved G*** 1.00 mm to (169.5, 56.5)
- moved G*** 1.00 mm to (163.5, 56.0)
- moved G*** 0.50 mm to (163.5, 49.5)
Other:
- board text added: "N0PAD V3.1415926535"
Changed lines of the file:
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@@
 			(drillshape 0)
 			(scaleselection 1)
-			(outputdirectory "C:/Users/vinic/Downloads/")
+			(outputdirectory "gerbers/")
 		)
 	)
@@
 	(footprint "assets:automatons"
 		(layer "F.Cu")
-		(at 158.5 57)
+		(at 158.5 56)
 		(property "Reference" "G***"
 			(at 0 0 0)
@@
 	(footprint "assets:illuminate"
 		(layer "F.Cu")
-		(at 169.5 57.5)
+		(at 169.5 56.5)
 		(property "Reference" "G***"
 			(at 0 0 0)
@@
 	(footprint "assets:super-earth"
 		(layer "F.Cu")
-		(at 163.5 50)
+		(at 163.5 49.5)
 		(property "Reference" "G***"
 			(at 0 0 0)
@@
 	(footprint "assets:terminids"
 		(layer "F.Cu")
-		(at 163.5 57)
+		(at 163.5 56)
 		(property "Reference" "G***"
 			(at 0 0 0)
@@
 		)
 	)
+	(gr_text "N0PAD V3.1415926535"
+		(at 155 60.5 0)
+		(layer "F.SilkS")
+		(effects
+			(font
+				(size 1 1)
+				(thickness 0.1)
+			)
+			(justify left bottom)
+		)
+	)
