File: hackpads/gpad/right/pcb/right.kicad_pcb (KiCad board)
At the start: 2 copper layers, 57.2 x 40.1 mm, 5 parts, among them U1 XIAO-RP2040-DIP

Commit message: improve to standard
Other:
- board text added: "XIAO HERE"
- board text added: "gpad"
Changed lines of the file:
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@@
 			(outputformat 1)
 			(mirror no)
-			(drillshape 1)
+			(drillshape 0)
 			(scaleselection 1)
-			(outputdirectory "")
+			(outputdirectory "../../production/pcb/")
 		)
 	)
@@
 		(layer "Edge.Cuts")
 	)
+	(gr_text "XIAO HERE"
+		(at 118 76 0)
+		(layer "B.SilkS")
+		(effects
+			(font
+				(size 1 1)
+				(thickness 0.1)
+			)
+			(justify left bottom mirror)
+		)
+	)
+	(gr_text "gpad"
+		(at 86.5 62 0)
+		(layer "F.SilkS")
+		(effects
+			(font
+				(size 1 1)
+				(thickness 0.1)
+			)
+			(justify left bottom)
+		)
+	)
 	(segment
