File: hackpads/Sammie's Chonkpad/PCB/hackpad.kicad_pcb (KiCad board)
At the start: 2 copper layers, 83.3 x 101.1 mm, 35 parts, among them SW1 SW_Push, SW10 SW_Push, SW11 SW_Push, SW12 SW_Push, SW13 SW_Push, SW14 SW_Push, SW15 SW_Push, SW16 SW_Push, SW2 SW_Push, SW3 SW_Push, SW4 SW_Push, SW5 SW_Push, SW6 SW_Push, SW7 SW_Push, SW8 SW_Push, SW9 SW_Push, U1 XIAO-RP2040-DIP

Commit message: Add files via upload
Other:
- board text added: "Sammie's Scarapad"
- board text removed: "Sammie's Chonkpad"
Changed lines of the file:
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@@
 		(layer "Edge.Cuts")
 	)
-	(gr_text "Sammie's Chonkpad"
+	(gr_text "Sammie's Scarapad"
 		(at 61.9125 42.8625 0)
 		(layer "F.SilkS")
