File: hackpads/Stoopid_pad/PCB/Hackpad!.kicad_pcb (KiCad board)
At the start: 2 copper layers, 100 x 69.3 mm, 16 parts, among them SW1 SW_Push, SW10 SW_Push, SW2 SW_Push, SW3 SW_Push, SW4 SW_Push, SW5 SW_Push, SW6 SW_Push, SW7 RotaryEncoder_Switch, SW9 SW_Push, U1 XIAO-RP2040-DIP, U2 MCP23017_SO

Commit message: Add files via upload
Other:
- board text added: "Stoopid_Pad :3"
Changed lines of the file:
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@@
 		(layer "Edge.Cuts")
+	)
+	(gr_text "Stoopid_Pad :3"
+		(at 147.6375 142.875 0)
+		(layer "Edge.Cuts")
+		(effects
+			(font
+				(size 1 1)
+				(thickness 0.15)
+			)
+			(justify left bottom)
+		)
 	)
 	(dimension
