File: hackpads/bacons hackpad/PCB/hackpad-final.kicad_pcb (KiCad board)
At the start: 2 copper layers, 82.5 x 61.5 mm, 19 parts, among them J1 OLED DISPLAY, SW1 SW_Push_45deg, SW2 SW_Push_45deg, SW3 SW_Push_45deg, SW4 SW_Push_45deg, SW5 SW_Push_45deg, SW6 SW_Push_45deg, SW7 RotaryEncoder_Switch, SW8 RotaryEncoder_Switch, U1 XIAO-RP2040-DIP

Commit message: Add files via upload
Other:
- board text added: "Baconpad"
