File: hackpads/endpad/endpad-pcb/hackpad.kicad_pcb (KiCad board)
At the start: 2 copper layers, 98.7 x 80.7 mm, 23 parts, among them SW1 SW_Push, SW10 SW_Push, SW11 SW_Push, SW12 SW_Push, SW13 SW_Push, SW14 SW_Push, SW15 SW_Push, SW16 SW_Push, SW2 SW_Push, SW3 SW_Push, SW4 SW_Push, SW5 SW_Push, SW6 RotaryEncoder_Switch, SW7 SW_Push, SW8 SW_Push, SW9 SW_Push, U1 XIAO-RP2040-DIP, U2 MCP23017_SO

Commit message: renamed and changed shit
Other:
- board text added: "A ProtoFox's Endpad Media Controller F13-24 V1"
- board text removed: "End's Foxpad Media Controller F13-24 V1"
Changed lines of the file:
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@@
 		)
 	)
-	(gr_text "End's Foxpad\nMedia Controller\nF13-24\nV1"
-		(at 159.4 148.4 0)
+	(gr_text "A ProtoFox's Endpad\nMedia Controller\nF13-24\nV1"
+		(at 157.5 148.5 0)
 		(layer "F.SilkS")
 		(effects

Commit message: o
Routing:
- net Net-(U2-GPA5): track 77.5 -> 75.8 mm
- net Net-(U1-GPIO0/TX): track 102.5 -> 101.5 mm
- net Net-(U1-GPIO4/MISO): track 61.7 -> 60.7 mm
- net ENC-B: track 154.0 -> 153.2 mm
- net Net-(U1-GPIO2/SCK): track 75.6 -> 75.0 mm

Commit message: .
Parts:
- G***: footprint LOGO -> 3D Models:LOGO
- moved SW15 2.38 mm to (116.8, 133.0)
- moved R2 2.38 mm to (145.3, 139.5)
- moved SW16 2.38 mm to (135.9, 133.0)
- moved R1 1.64 mm to (147.6, 139.5)
Routing:
- net Net-(U2-GPB6): track 38.0 -> 98.5 mm, vias 3 -> 1
- net Net-(U1-GPIO7/SCL): track 99.3 -> 114.6 mm
- net Net-(U1-GPIO0/TX): track 101.5 -> 93.3 mm, vias 2 -> 0
- net +3.3V: track 116.9 -> 109.9 mm
- net GND: track 351.3 -> 355.8 mm, vias 0 -> 1
- net Net-(U2-GPB5): track 32.9 -> 37.0 mm
- net Net-(U2-GPB4): track 52.7 -> 49.1 mm
- net Net-(U2-GPB3): track 30.5 -> 28.1 mm
Other:
- board text added: "IO EXPANDER HERE"
