File: hackpads/endpad/endpad-pcb/hackpad3d.kicad_sch (KiCad schematic)
At the start: 22 parts, among them SW1 SW_Push, SW10 SW_Push, SW11 SW_Push, SW12 SW_Push, SW13 SW_Push, SW14 SW_Push, SW15 SW_Push, SW16 SW_Push, SW2 SW_Push, SW3 SW_Push, SW4 SW_Push, SW5 SW_Push, SW6 RotaryEncoder_Switch, SW7 SW_Push, SW8 SW_Push, SW9 SW_Push, U1 XIAO-RP2040-DIP, U2 MCP23017_SO

Commit message: o
Changed lines of the file:
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@@
 (kicad_sch
-	(version 20231120)
+	(version 20250114)
 	(generator "eeschema")
-	(generator_version "8.0")
+	(generator_version "9.0")
 	(paper "A4")
+	(text "F16"
+		(exclude_from_sim no)
+		(at 50.292 101.6 0)
+		(effects
+			(font
+				(size 1.27 1.27)
+			)
+		)
+	)
+	(text "F18\n"
+		(exclude_from_sim no)
+		(at 50.8 106.934 0)
+		(effects
+			(font
+				(size 1.27 1.27)
+			)
+		)
+	)
+	(text "F13"
+		(exclude_from_sim no)
+		(at 53.086 135.636 0)
+		(effects
+			(font
+				(size 1.27 1.27)
+			)
+		)
+	)
+	(text "F17"
+		(exclude_from_sim no)
+		(at 48.768 116.078 0)
+		(effects
+			(font
+				(size 1.27 1.27)
+			)
+		)
+	)
+	(text "F23"
+		(exclude_from_sim no)
+		(at 23.622 113.792 0)
+		(effects
+			(font
+				(size 1.27 1.27)
+			)
+		)
+	)
+	(text "Volume Knob/Mute Switch"
+		(exclude_from_sim no)
+		(at 56.642 171.196 0)
+		(effects
+			(font
+				(size 1.27 1.27)
+			)
+		)
+	)
+	(text "F19"
+		(exclude_from_sim no)
+		(at 52.07 97.536 0)
+		(effects
+			(font
+				(size 1.27 1.27)
+			)
+		)
+	)
+	(text "Skip Forward"
+		(exclude_from_sim no)
+		(at 54.61 145.034 0)
+		(effects
+			(font
+				(size 1.27 1.27)
+			)
+		)
+	)
+	(text "F20"
+		(exclude_from_sim no)
+		(at 49.276 125.222 0)
+		(effects
+			(font
+				(size 1.27 1.27)
+			)
+		)
+	)
+	(text "F22"
+		(exclude_from_sim no)
+		(at 23.114 102.616 0)
+		(effects
+			(font
+				(size 1.27 1.27)
+			)
+		)
+	)
+	(text "F24"
+		(exclude_from_sim no)
+		(at 24.13 127 0)
+		(effects
+			(font
+				(size 1.27 1.27)
+			)
+		)
+	)
+	(text "F15"
+		(exclude_from_sim no)
+		(at 50.546 112.268 0)
+		(effects
+			(font
+				(size 1.27 1.27)
+			)
+		)
+	)
+	(text "Skip Back"
+		(exclude_from_sim no)
+		(at 52.832 154.94 0)
+		(effects
+			(font
+				(size 1.27 1.27)
+			)
+		)
+	)
+	(text "F21"
+		(exclude_from_sim no)
+		(at 59.436 133.858 0)
+		(effects
+			(font
+				(size 1.27 1.27)
+			)
+		)
+	)
+	(text "Play/Pause Switch"
+		(exclude_from_sim no)
+		(at 56.642 165.354 0)
+		(effects
+			(font
+				(size 1.27 1.27)
+			)
+		)
+	)
+	(text "F14\n"
+		(exclude_from_sim no)
+		(at 50.8 123.444 0)
+		(effects
+			(font
+				(size 1.27 1.27)
+			)
+		)
+	)
 	(junction
 		(at 123.19 69.85)
@@
 		)
 	)
-	(text "F16"
-		(exclude_from_sim no)
-		(at 50.292 101.6 0)
-		(effects
-			(font
-				(size 1.27 1.27)
-			)
-		)
-	)
-	(text "F18\n"
-		(exclude_from_sim no)
-		(at 50.8 106.934 0)
-		(effects
-			(font
-				(size 1.27 1.27)
-			)
-		)
-	)
-	(text "F13"
-		(exclude_from_sim no)
-		(at 53.086 135.636 0)
-		(effects
-			(font
-				(size 1.27 1.27)
-			)
-		)
-	)
-	(text "F17"
-		(exclude_from_sim no)
-		(at 48.768 116.078 0)
-		(effects
-			(font
-				(size 1.27 1.27)
-			)
-		)
-	)
-	(text "F23"
-		(exclude_from_sim no)
-		(at 23.622 113.792 0)
-		(effects
-			(font
-				(size 1.27 1.27)
-			)
-		)
-	)
-	(text "Volume Knob/Mute Switch"
-		(exclude_from_sim no)
-		(at 56.642 171.196 0)
-		(effects
-			(font
-				(size 1.27 1.27)
-			)
-		)
-	)
-	(text "F19"
-		(exclude_from_sim no)
-		(at 52.07 97.536 0)
-		(effects
-			(font
-				(size 1.27 1.27)
-			)
-		)
-	)
-	(text "Skip Forward"
-		(exclude_from_sim no)
-		(at 54.61 145.034 0)
-		(effects
-			(font
-				(size 1.27 1.27)
-			)
-		)
-	)
-	(text "F20"
-		(exclude_from_sim no)
-		(at 49.276 125.222 0)
-		(effects
-			(font
-				(size 1.27 1.27)
-			)
-		)
-	)
-	(text "F22"
-		(exclude_from_sim no)
-		(at 23.114 102.616 0)
-		(effects
-			(font
-				(size 1.27 1.27)
-			)
-		)
-	)
-	(text "F24"
-		(exclude_from_sim no)
-		(at 24.13 127 0)
-		(effects
-			(font
-				(size 1.27 1.27)
-			)
-		)
-	)
-	(text "F15"
-		(exclude_from_sim no)
-		(at 50.546 112.268 0)
-		(effects
-			(font
-				(size 1.27 1.27)
-			)
-		)
-	)
-	(text "Skip Back"
-		(exclude_from_sim no)
-		(at 52.832 154.94 0)
-		(effects
-			(font
-				(size 1.27 1.27)
-			)
-		)
-	)
-	(text "F21"
-		(exclude_from_sim no)
-		(at 59.436 133.858 0)
-		(effects
-			(font
-				(size 1.27 1.27)
-			)
-		)
-	)
-	(text "Play/Pause Switch"
-		(exclude_from_sim no)
-		(at 56.642 165.354 0)
-		(effects
-			(font
-				(size 1.27 1.27)
-			)
-		)
-	)
-	(text "F14\n"
-		(exclude_from_sim no)
-		(at 50.8 123.444 0)
-		(effects
-			(font
-				(size 1.27 1.27)
-			)
-		)
-	)
 	(global_label "ENC-A"
 		(shape input)
@@
 		)
 	)
+	(embedded_fonts no)
 )

Commit message: .
Parts:
- R1, R2: footprint Resistor_THT:R_Axial_DIN0204_L3.6mm_D1.6mm_P7.62mm_Horizontal -> 3D Models:R_Axial_DIN0204_L3.6mm_D1.6mm_P7.62mm_Horizontal
Changed lines of the file:
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@@
 			)
 		)
-		(property "Footprint" "Resistor_THT:R_Axial_DIN0204_L3.6mm_D1.6mm_P7.62mm_Horizontal"
+		(property "Footprint" "3D Models:R_Axial_DIN0204_L3.6mm_D1.6mm_P7.62mm_Horizontal"
 			(at 22.352 25.4 90)
 			(effects
@@
 			)
 		)
-		(property "Footprint" "Resistor_THT:R_Axial_DIN0204_L3.6mm_D1.6mm_P7.62mm_Horizontal"
+		(property "Footprint" "3D Models:R_Axial_DIN0204_L3.6mm_D1.6mm_P7.62mm_Horizontal"
 			(at 29.972 25.4 90)
 			(effects
