File: hackpads/endpad/endpad-pcb/hackpad3d.kicad_pcb (KiCad board)
At the start: 2 copper layers, 98.7 x 80.7 mm, 23 parts, among them SW1 SW_Push, SW10 SW_Push, SW11 SW_Push, SW12 SW_Push, SW13 SW_Push, SW14 SW_Push, SW15 SW_Push, SW16 SW_Push, SW2 SW_Push, SW3 SW_Push, SW4 SW_Push, SW5 SW_Push, SW6 RotaryEncoder_Switch, SW7 SW_Push, SW8 SW_Push, SW9 SW_Push, U1 XIAO-RP2040-DIP, U2 MCP23017_SO

Commit message: renamed and changed shit
Other:
- board text added: "A ProtoFox's Endpad Media Controller F13-24 V1"
- board text removed: "End's Foxpad Media Controller F13-24 V1"
Changed lines of the file:
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@@
 		)
 	)
-	(gr_text "End's Foxpad\nMedia Controller\nF13-24\nV1"
-		(at 159.4 148.4 0)
+	(gr_text "A ProtoFox's Endpad\nMedia Controller\nF13-24\nV1"
+		(at 157 148.75 0)
 		(layer "F.SilkS")
 		(effects

Commit message: o
Parts:
- G***: footprint LOGO -> 3D Models:LOGO
Routing:
- net Net-(U2-GPA5): track 77.5 -> 75.8 mm
- net Net-(U1-GPIO0/TX): track 102.5 -> 101.5 mm
- net Net-(U1-GPIO4/MISO): track 61.7 -> 60.7 mm
- net ENC-B: track 154.0 -> 153.2 mm
- net Net-(D1-DIN): track 126.8 -> 127.5 mm
- net Net-(U1-GPIO2/SCK): track 75.6 -> 75.0 mm

Commit message: .
Parts:
- R1, R2: footprint Resistor_THT:R_Axial_DIN0204_L3.6mm_D1.6mm_P7.62mm_Horizontal -> 3D Models:R_Axial_DIN0204_L3.6mm_D1.6mm_P7.62mm_Horizontal
- moved SW15 2.38 mm to (116.8, 133.0)
- moved R2 2.38 mm to (145.3, 139.5)
- moved SW16 2.38 mm to (135.9, 133.0)
- moved R1 1.64 mm to (147.6, 139.5)
Routing:
- net Net-(U2-GPB6): track 38.0 -> 98.5 mm, vias 3 -> 1
- net Net-(U1-GPIO7/SCL): track 99.3 -> 114.6 mm
- net Net-(U1-GPIO0/TX): track 101.5 -> 93.3 mm, vias 2 -> 0
- net +3.3V: track 116.9 -> 109.9 mm
- net GND: track 351.3 -> 355.8 mm, vias 0 -> 1
- net Net-(U2-GPB5): track 32.9 -> 37.0 mm
- net Net-(U2-GPB4): track 52.7 -> 49.1 mm
- net Net-(U2-GPB3): track 30.5 -> 28.1 mm

Commit message: .
Other:
- board text added: "A ProtoFox's Endpad V1"
- board text removed: "A ProtoFox's Endpad Media Controller F13-24 V1"
Changed lines of the file:
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@@
 		(tags "Resistor Axial_DIN0204 series Axial Horizontal pin pitch 7.62mm 0.167W length 3.6mm diameter 1.6mm")
 		(property "Reference" "R1"
-			(at 3.81 -1.92 90)
+			(at -2 -0.1375 90)
 			(layer "F.SilkS")
 			(effects
@@
 			(at 3.81 1.92 90)
 			(layer "F.Fab")
+			(hide yes)
 			(effects
 				(font
@@
 	(footprint "3D Models:R_Axial_DIN0204_L3.6mm_D1.6mm_P7.62mm_Horizontal"
 		(layer "F.Cu")
-		(at 145.25625 139.54125 90)
+		(at 145.25625 139.5 90)
 		(descr "Resistor, Axial_DIN0204 series, Axial, Horizontal, pin pitch=7.62mm, 0.167W, length*diameter=3.6*1.6mm^2, http://cdn-reichelt.de/documents/datenblatt/B400/1_4W%23YAG.pdf")
 		(tags "Resistor Axial_DIN0204 series Axial Horizontal pin pitch 7.62mm 0.167W length 3.6mm diameter 1.6mm")
 		(property "Reference" "R2"
-			(at 3.81 -1.92 90)
+			(at -1.95875 -0.25625 90)
 			(layer "F.SilkS")
 			(effects
@@
 			(at 3.81 1.92 90)
 			(layer "F.Fab")
+			(hide yes)
 			(effects
 				(font
@@
 			)
 		)
-		(property "Datasheet" "https://ww1.microchip.com/downloads/aemDocuments/documents/APID/ProductDocuments/DataSheets/MCP23017-Data-Sheet-DS20001952.pdf"
+		(property "Datasheet" ""
 			(at 0 0 90)
 			(layer "F.Fab")
@@
 			)
 		)
-		(property "Description" "16-bit I/O expander, I2C, interrupts, w pull-ups, GPA/B7 output only (https://microchip.my.site.com/s/article/GPA7---GPB7-Cannot-Be-Used-as-Inputs-In-MCP23017),  SOIC-28"
+		(property "Description" ""
 			(at 0 0 90)
 			(layer "F.Fab")
@@
 		(at 85.725 138.1125 90)
 		(property "Reference" "U1"
-			(at -8.5 -12 90)
+			(at 0.1125 10.775 90)
 			(unlocked yes)
 			(layer "F.SilkS")
@@
 		(sheetname "/")
 		(sheetfile "hackpad.kicad_sch")
-		(attr smd)
+		(attr through_hole)
 		(fp_line
 			(start -3.991272 -11.951)
@@
 		)
 		(embedded_fonts no)
-		(model "${AMZPATH}/3dmodels/AMz3D.3dshapes/XIAO-nRF52840 v15.step"
-			(hide yes)
-			(offset
-				(xyz -1.778 -6.096 0.381)
-			)
-			(scale
-				(xyz 1 1 1)
-			)
-			(rotate
-				(xyz -90 0 0)
-			)
-		)
-		(model "${AMZPATH}/3dmodels/AMz3D.3dshapes/Seeeduino XIAO SAMD21 v4.step"
-			(hide yes)
-			(offset
-				(xyz 0 0 0)
-			)
-			(scale
-				(xyz 1 1 1)
-			)
-			(rotate
-				(xyz 0 0 0)
-			)
-		)
-		(model "${AMZPATH}/3dmodels/AMz3D.3dshapes/Seeed Studio XIAO RP2040 v26.step"
-			(hide yes)
-			(offset
-				(xyz 0 0 0)
-			)
-			(scale
-				(xyz 1 1 1)
-			)
-			(rotate
-				(xyz 0 0 90)
-			)
-		)
-		(model "${AMZPATH}/3dmodels/AMz3D.3dshapes/Seeed Studio XIAO-ESP32-C3.step"
-			(hide yes)
-			(offset
-				(xyz -1.7018 -6.096 0)
-			)
-			(scale
-				(xyz 1 1 1)
-			)
-			(rotate
-				(xyz -90 0 0)
-			)
-		)
-		(model "${AMZPATH}/3dmodels/AMz3D.3dshapes/XIAO-ESP32S3 v2.step"
-			(hide yes)
-			(offset
-				(xyz -1.778 -6.1722 0)
-			)
-			(scale
-				(xyz 1 1 1)
-			)
-			(rotate
-				(xyz -90 0 0)
-			)
-		)
 		(model "${KIPRJMOD}/3D Models.pretty/Seeed Studio XIAO RP2040 v26.step"
 			(offset
@@
 		)
 	)
-	(gr_text "A ProtoFox's Endpad\nMedia Controller\nF13-24\nV1"
+	(gr_text "A ProtoFox's Endpad\nV1"
 		(at 157.5 148.5 0)
 		(layer "F.SilkS")
