File: hackboards/CherryTree56567_Keyboard/pcb/pcb.kicad_pcb (KiCad board)
At the start: 2 copper layers, 284.6 x 110.1 mm, 152 parts, among them J1 USB_C_Receptacle_USB2.0, J2 USB_C_Receptacle_USB2.0, J4 USB_C_Receptacle_USB2.0, J5 USB_C_Receptacle_USB2.0, J6 PGA2040, SW3 RESET, SW4 BOOTSEL, U1 SL2.1A

Commit message: Modify the thing to use RP2040
Parts:
- removed J6: PGA2040, footprints:PGA2040_PTH_NO_SLOT
- removed SW3: RESET, Button_Switch_SMD:SW_Push_1P1T_NO_Vertical_Wuerth_434133025816
- removed SW4: BOOTSEL, Button_Switch_SMD:SW_Push_1P1T_NO_Vertical_Wuerth_434133025816
- added C1: 15p, Capacitor_SMD:C_0402_1005Metric, F.Cu at (208.5, 111.1)
- added C10: 1u, Capacitor_SMD:C_0402_1005Metric, F.Cu at (202.5, 111.1)
- added C11: 100n, Capacitor_SMD:C_0402_1005Metric, F.Cu at (202.5, 109.9)
- added C12: 100n, Capacitor_SMD:C_0402_1005Metric, F.Cu at (201.3, 108.8)
- added C13: 100n, Capacitor_SMD:C_0402_1005Metric, F.Cu at (221.6, 109.9)
- added C14: 100n, Capacitor_SMD:C_0402_1005Metric, F.Cu at (224.0, 111.1)
- added C15: 100n, Capacitor_SMD:C_0402_1005Metric, F.Cu at (218.5, 114.7)
- added C16: 100n, Capacitor_SMD:C_0402_1005Metric, F.Cu at (224.4, 114.7)
- added C2: 15p, Capacitor_SMD:C_0402_1005Metric, F.Cu at (208.5, 112.3)
- added C3: 10u, Capacitor_SMD:C_0805_2012Metric, F.Cu at (184.2, 107.6)
- added C4: 10u, Capacitor_SMD:C_0805_2012Metric, F.Cu at (222.3, 107.6)
- added C5: 100n, Capacitor_SMD:C_0402_1005Metric, F.Cu at (200.6, 109.9)
- added C6: 100n, Capacitor_SMD:C_0402_1005Metric, F.Cu at (221.3, 112.3)
- added C7: 100n, Capacitor_SMD:C_0402_1005Metric, F.Cu at (221.6, 111.1)
- added C8: 1u, Capacitor_SMD:C_0402_1005Metric, F.Cu at (224.0, 109.9)
- added C9: 100n, Capacitor_SMD:C_0402_1005Metric, F.Cu at (224.0, 112.3)
- added R3: 1k, Resistor_SMD:R_0402_1005Metric, F.Cu at (201.3, 114.7)
- added R4: DNF, Resistor_SMD:R_0402_1005Metric, F.Cu at (188.2, 107.6)
- added R5: 1k, Resistor_SMD:R_0402_1005Metric, F.Cu at (203.7, 114.7)
- added R6: 27, Resistor_SMD:R_0402_1005Metric, B.Cu at (184.6, 195.7)
- added R7: 27, Resistor_SMD:R_0402_1005Metric, B.Cu at (187.0, 195.7)
- added SW1: SW_Push, Button_Switch_SMD:SW_Push_1P1T_NO_Vertical_Wuerth_434133025816, B.Cu at (199.4, 199.2)
- added U2: NCP1117-3.3_SOT223, Package_TO_SOT_SMD:SOT-223-3_TabPin2, F.Cu at (215.7, 110.0)
- added U3: W25Q128JVS, Package_SO:SOIC-8_5.23x5.23mm_P1.27mm, F.Cu at (194.6, 111.1)
- added U4: RP2040, RP2040_minimal_r2:RP2040-QFN-56, B.Cu at (179.2, 200.4)
- added Y1: ABM8-272-T3, Crystal:Crystal_SMD_3225-4Pin_3.2x2.5mm, F.Cu at (207.9, 107.9)
Connections:
- net /USBC_VBUS renamed VBUS
Routing:
- net +3V3: track 0.00 -> 224.1 mm, vias 0 -> 5
- net +1V1: track 0.00 -> 167.8 mm, vias 0 -> 7
- net VBUS: track 380.8 -> 215.5 mm, vias 11 -> 5
- net /XIN: track 0.00 -> 156.6 mm, vias 0 -> 5
- net /~{USB_BOOT}: track 0.00 -> 145.1 mm, vias 0 -> 3
- net /QSPI_SD3: track 0.00 -> 143.3 mm, vias 0 -> 5
- net /QSPI_SS: track 0.00 -> 140.0 mm, vias 0 -> 5
- net /XOUT: track 0.00 -> 138.9 mm, vias 0 -> 5
- net /QSPI_SCLK: track 0.00 -> 127.0 mm, vias 0 -> 5
- net /QSPI_SD2: track 0.00 -> 122.4 mm, vias 0 -> 5
- net /QSPI_SD0: track 0.00 -> 119.0 mm, vias 0 -> 5
- net /QSPI_SD1: track 0.00 -> 108.5 mm, vias 0 -> 5
- net USBC_GND: track 533.6 -> 599.3 mm, vias 3 -> 8
- net Net-(J6-BOOTSEL): track 40.3 -> 0.00 mm, vias 2 -> 0
- net row2: track 461.6 -> 428.3 mm
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